File: Kicad/Rotonometron_PCB/Rotonometron_PCB.kicad_sch (KiCad schematic)
At the start: 145 parts, among them J1 JOYSTICK_SLIDE, P1 Pin_R, P10 Pin_R, P11 Pin_R, P2 Pin_S, P3 Pin_R, P4 Pin_R, P5 Pin_R, P6 Pin_R, P7 Pin_S, P8 Pin_R, P9 Pin_S, SW1 HECKIN_LED_SWITCH, SW10 HECKIN_LED_SWITCH, SW11 HECKIN_LED_SWITCH, SW12 HECKIN_LED_SWITCH, SW13 HECKIN_LED_SWITCH, SW14 HECKIN_LED_SWITCH, SW15 HECKIN_LED_SWITCH, SW16 HECKIN_LED_SWITCH, SW17 HECKIN_LED_SWITCH, SW18 HECKIN_LED_SWITCH, SW19 HECKIN_LED_SWITCH, SW2 HECKIN_LED_SWITCH, SW20 HECKIN_LED_SWITCH, SW21 HECKIN_LED_SWITCH, SW22 HECKIN_LED_SWITCH, SW23 HECKIN_LED_SWITCH, SW24 HECKIN_LED_SWITCH, SW25 HECKIN_LED_SWITCH, SW26 HECKIN_LED_SWITCH, SW27 HECKIN_LED_SWITCH, SW28 HECKIN_LED_SWITCH, SW29 HECKIN_LED_SWITCH, SW3 HECKIN_LED_SWITCH, SW30 HECKIN_LED_SWITCH, SW31 HECKIN_LED_SWITCH, SW32 HECKIN_LED_SWITCH, SW33 HECKIN_LED_SWITCH, SW34 HECKIN_LED_SWITCH, SW35 HECKIN_LED_SWITCH, SW36 HECKIN_LED_SWITCH, SW37 HECKIN_LED_SWITCH, SW38 HECKIN_LED_SWITCH, SW4 HECKIN_LED_SWITCH, SW5 HECKIN_LED_SWITCH, SW6 HECKIN_LED_SWITCH, SW7 HECKIN_LED_SWITCH, SW8 HECKIN_LED_SWITCH, SW9 HECKIN_LED_SWITCH, U1 PCA9506BS,118, U2 PCA9506BS,118, U3 XIAOBLE

Commit message: forked V2
Parts:
- SW1, SW10, SW11, SW12, SW13, SW14, SW15, SW16, SW17, SW18, SW19, SW2, SW20, SW21, SW22, SW23, SW24, SW25, SW26, SW27, SW28, SW29, SW3, SW30, SW31, SW32, SW33, SW34, SW35, SW36, SW37, SW38, SW4, SW5, SW6, SW7, SW8, SW9: value HECKIN_LED_SWITCH -> Heckin_LED_Switch; symbol Universal_Keyswitch:HECKIN_LED_SWITCH -> Custom:Heckin_LED_Switch
Connections:
- net +5V: now also SW1.5v, SW10.5v, SW11.5v, SW12.5v, SW13.5v, SW14.5v, SW15.5v, SW16.5v, SW17.5v, SW18.5v, SW19.5v, SW2.5v, SW20.5v, SW21.5v, SW22.5v, SW23.5v, SW24.5v, SW25.5v, SW26.5v, SW27.5v, SW28.5v, SW29.5v, SW3.5v, SW30.5v, SW31.5v, SW32.5v, SW33.5v, SW34.5v, SW35.5v, SW36.5v, SW37.5v, SW38.5v, SW4.5v, SW5.5v, SW6.5v, SW7.5v, SW8.5v, SW9.5v; no longer SW1.3 (5v), SW10.3 (5v), SW11.3 (5v), SW12.3 (5v), SW13.3 (5v), SW14.3 (5v), SW15.3 (5v), SW16.3 (5v), SW17.3 (5v), SW18.3 (5v), SW19.3 (5v), SW2.3 (5v), SW20.3 (5v), SW21.3 (5v), SW22.3 (5v), SW23.3 (5v), SW24.3 (5v), SW25.3 (5v), SW26.3 (5v), SW27.3 (5v), SW28.3 (5v), SW29.3 (5v), SW3.3 (5v), SW30.3 (5v), SW31.3 (5v), SW32.3 (5v), SW33.3 (5v), SW34.3 (5v), SW35.3 (5v), SW36.3 (5v), SW37.3 (5v), SW38.3 (5v), SW4.3 (5v), SW5.3 (5v), SW6.3 (5v), SW7.3 (5v), SW8.3 (5v), SW9.3 (5v)
- net GND: now also SW1.GND, SW10.GND, SW11.GND, SW12.GND, SW13.GND, SW14.GND, SW15.GND, SW16.GND, SW17.GND, SW18.GND, SW19.GND, SW2.GND, SW20.GND, SW21.GND, SW22.GND, SW23.GND, SW24.GND, SW25.GND, SW26.GND, SW27.GND, SW28.GND, SW29.GND, SW3.GND, SW30.GND, SW31.GND, SW32.GND, SW33.GND, SW34.GND, SW35.GND, SW36.GND, SW37.GND, SW38.GND, SW4.GND, SW5.GND, SW6.GND, SW7.GND, SW8.GND, SW9.GND; no longer SW1.6 (GND), SW10.6 (GND), SW11.6 (GND), SW12.6 (GND), SW13.6 (GND), SW14.6 (GND), SW15.6 (GND), SW16.6 (GND), SW17.6 (GND), SW18.6 (GND), SW19.6 (GND), SW2.6 (GND), SW20.6 (GND), SW21.6 (GND), SW22.6 (GND), SW23.6 (GND), SW24.6 (GND), SW25.6 (GND), SW26.6 (GND), SW27.6 (GND), SW28.6 (GND), SW29.6 (GND), SW3.6 (GND), SW30.6 (GND), SW31.6 (GND), SW32.6 (GND), SW33.6 (GND), SW34.6 (GND), SW35.6 (GND), SW36.6 (GND), SW37.6 (GND), SW38.6 (GND), SW4.6 (GND), SW5.6 (GND), SW6.6 (GND), SW7.6 (GND), SW8.6 (GND), SW9.6 (GND)
- net LED control: now also SW1.DIN; no longer SW1.5 (DIN)
- net at LED1.2 (DIN): now also SW38.DOUT; no longer SW38.4 (DOUT)
- new net: SW2.DOUT, SW3.DIN
- new net: SW3.DOUT, SW4.DIN
- new net: SW27.DOUT, SW28.DIN
- new net: SW28.DOUT, SW29.DIN
- new net: SW17.DOUT, SW18.DIN
- new net: SW18.DOUT, SW19.DIN
- new net: SW10.DOUT, SW11.DIN
- new net: SW11.DOUT, SW12.DIN
- new net: SW26.DOUT, SW27.DIN
- new net: SW35.DOUT, SW36.DIN
- new net: SW36.DOUT, SW37.DIN
- new net: SW1.DOUT, SW2.DIN
- new net: SW5.DOUT, SW6.DIN
- new net: SW6.DOUT, SW7.DIN
- new net: SW10.DIN, SW9.DOUT
- new net: SW23.DOUT, SW24.DIN
- new net: SW24.DOUT, SW25.DIN
- new net: SW31.DOUT, SW32.DIN
- new net: SW32.DOUT, SW33.DIN
- new net: SW15.DOUT, SW16.DIN
- new net: SW16.DOUT, SW17.DIN
- new net: SW30.DOUT, SW31.DIN
- new net: SW7.DOUT, SW8.DIN
- new net: SW37.DOUT, SW38.DIN
- new net: SW25.DOUT, SW26.DIN
- new net: SW13.DOUT, SW14.DIN
- new net: SW14.DOUT, SW15.DIN
- new net: SW19.DOUT, SW20.DIN
- new net: SW21.DOUT, SW22.DIN
- new net: SW22.DOUT, SW23.DIN
- new net: SW34.DOUT, SW35.DIN
- new net: SW12.DOUT, SW13.DIN
- new net: SW4.DOUT, SW5.DIN
- new net: SW33.DOUT, SW34.DIN
- new net: SW8.DOUT, SW9.DIN
- new net: SW20.DOUT, SW21.DIN
- new net: SW29.DOUT, SW30.DIN
