File: Kicad/Rotonometron_PCB_rev2/Rotonometron_V2/Rotonometron_V2.kicad_sch (KiCad schematic)
At the start: 145 parts, among them J1 JOYSTICK_SLIDE, P1 Pin_R, P10 Pin_R, P11 Pin_R, P2 Pin_S, P3 Pin_R, P4 Pin_R, P5 Pin_R, P6 Pin_R, P7 Pin_S, P8 Pin_R, P9 Pin_S, SW1 Heckin_LED_Switch, SW10 Heckin_LED_Switch, SW11 Heckin_LED_Switch, SW12 Heckin_LED_Switch, SW13 Heckin_LED_Switch, SW14 Heckin_LED_Switch, SW15 Heckin_LED_Switch, SW16 Heckin_LED_Switch, SW17 Heckin_LED_Switch, SW18 Heckin_LED_Switch, SW19 Heckin_LED_Switch, SW2 Heckin_LED_Switch, SW20 Heckin_LED_Switch, SW21 Heckin_LED_Switch, SW22 Heckin_LED_Switch, SW23 Heckin_LED_Switch, SW24 Heckin_LED_Switch, SW25 Heckin_LED_Switch, SW26 Heckin_LED_Switch, SW27 Heckin_LED_Switch, SW28 Heckin_LED_Switch, SW29 Heckin_LED_Switch, SW3 Heckin_LED_Switch, SW30 Heckin_LED_Switch, SW31 Heckin_LED_Switch, SW32 Heckin_LED_Switch, SW33 Heckin_LED_Switch, SW34 Heckin_LED_Switch, SW35 Heckin_LED_Switch, SW36 Heckin_LED_Switch, SW37 Heckin_LED_Switch, SW38 Heckin_LED_Switch, SW4 Heckin_LED_Switch, SW5 Heckin_LED_Switch, SW6 Heckin_LED_Switch, SW7 Heckin_LED_Switch, SW8 Heckin_LED_Switch, SW9 Heckin_LED_Switch, U1 PCA9506BS,118, U2 PCA9506BS,118, U3 XIAOBLE

Commit message: v2.01
Parts:
- removed U1, U2: PCA9506BS,118, NXP_Semiconductors-PCA9506BS,118-*, symbol eec:PCA9506BS,118
- added U1, U2: PCA9505DGG,118, PCA9505DGG_118:SOP50P810X120-56N, symbol PCA9505DGG_118:PCA9505DGG,118
- BT1: footprint BATTERY_18650-HOLDER -> Batteries:BATTERY_18650-HOLDER
Connections:
- new net: U1.11 (VSS), U1.23 (VSS), U1.34 (VSS), U1.39 (VSS), U1.51 (VSS), U1.6 (VSS)
- new net: U1.18 (VDD), U1.46 (VDD)
- new net: U2.11 (VSS), U2.23 (VSS), U2.34 (VSS), U2.39 (VSS), U2.51 (VSS), U2.6 (VSS)
- new net: U2.18 (VDD), U2.46 (VDD)

Commit message: .
Parts:
- removed R1, R10, R11, R12, R13, R14, R15, R16, R17, R18, R19, R2, R20, R21, R22, R23, R24, R25, R26, R27, R28, R29, R3, R30, R31, R32, R33, R34, R35, R36, R37, R38, R4, R5, R6, R7, R8, R9: 1kΩ, Resistor_SMD:R_0201_0603Metric_Pad0.64x0.40mm_HandSolder, symbol Device:R_Small
- added LED32, LED33, LED34, LED35, LED36: SK6812, Custom:Neopixel 2040, symbol SparkFun-DiscreteSemi:SK6812
- added U3: PCA9505DGG,118, PCA9505DGG_118:SOP50P810X120-56N, symbol PCA9505DGG_118:PCA9505DGG,118
- renumbered U3 to U4
Connections:
- net +5V: now also LED32.3 (VDD), LED33.3 (VDD), LED34.3 (VDD), LED35.3 (VDD), LED36.3 (VDD); no longer SW1.1 (Sw1), SW10.1 (Sw1), SW11.1 (Sw1), SW12.1 (Sw1), SW13.1 (Sw1), SW14.1 (Sw1), SW15.1 (Sw1), SW16.1 (Sw1), SW17.1 (Sw1), SW18.1 (Sw1), SW19.1 (Sw1), SW2.1 (Sw1), SW20.1 (Sw1), SW21.1 (Sw1), SW22.1 (Sw1), SW23.1 (Sw1), SW24.1 (Sw1), SW25.1 (Sw1), SW26.1 (Sw1), SW27.1 (Sw1), SW28.1 (Sw1), SW29.1 (Sw1), SW3.1 (Sw1), SW30.1 (Sw1), SW31.1 (Sw1), SW32.1 (Sw1), SW33.1 (Sw1), SW34.1 (Sw1), SW35.1 (Sw1), SW36.1 (Sw1), SW37.1 (Sw1), SW38.1 (Sw1), SW4.1 (Sw1), SW5.1 (Sw1), SW6.1 (Sw1), SW7.1 (Sw1), SW8.1 (Sw1), SW9.1 (Sw1)
- net GND: now also SW1.1 (Sw1), SW10.1 (Sw1), SW11.1 (Sw1), SW12.1 (Sw1), SW13.1 (Sw1), SW14.1 (Sw1), SW15.1 (Sw1), SW16.1 (Sw1), SW17.1 (Sw1), SW18.1 (Sw1), SW19.1 (Sw1), SW2.1 (Sw1), SW20.1 (Sw1), SW21.1 (Sw1), SW22.1 (Sw1), SW23.1 (Sw1), SW24.1 (Sw1), SW25.1 (Sw1), SW26.1 (Sw1), SW27.1 (Sw1), SW28.1 (Sw1), SW29.1 (Sw1), SW3.1 (Sw1), SW30.1 (Sw1), SW31.1 (Sw1), SW32.1 (Sw1), SW33.1 (Sw1), SW34.1 (Sw1), SW35.1 (Sw1), SW36.1 (Sw1), SW37.1 (Sw1), SW38.1 (Sw1), SW4.1 (Sw1), SW5.1 (Sw1), SW6.1 (Sw1), SW7.1 (Sw1), SW8.1 (Sw1), SW9.1 (Sw1), LED32.1 (VSS), LED33.1 (VSS), LED34.1 (VSS), LED35.1 (VSS), LED36.1 (VSS); no longer SW10.GND, SW11.GND, SW12.GND, SW13.GND, SW14.GND, SW8.GND, SW9.GND
- net RSw 0: now also U1.3 (IO0_0)
- net RSw 1: now also U1.7 (IO0_3)
- net Rot 0 A: now also U1.47 (IO4_1)
- net Rot 0 B: now also U1.45 (IO4_0)
- net Rot 0 G: now also U1.53 (IO4_6)
- net Rot 0 R: now also U1.52 (IO4_5)
- net Rot 0 U: now also U1.54 (IO4_7)
- net Rot 1 R: now also U1.4 (IO0_1)
- net Rot 1 U: now also U1.5 (IO0_2)
- net SCL: now also U1.2 (SCL), U2.2 (SCL), U3.2 (SCL)
- net SDA: now also U1.1 (SDA), U2.1 (SDA), U3.1 (SDA)
- net Sw 1: now also U1.44 (IO3_7)
- net Sw 10: now also U1.25 (IO2_2)
- net Sw 11: now also U1.15 (IO1_2)
- net Sw 15: now also U1.42 (IO3_5)
- net Sw 16: now also U1.33 (IO2_6)
- net Sw 17: now also U1.24 (IO2_1)
- net Sw 18: now also U1.16 (IO1_3)
- net Sw 2: now also U1.31 (IO2_4)
- net Sw 22: now also U1.41 (IO3_4)
- net Sw 23: now also U1.35 (IO2_7)
- net Sw 24: now also U1.22 (IO2_0)
- net Sw 25: now also U1.17 (IO1_4)
- net Sw 29: now also U1.40 (IO3_3)
- net Sw 3: now also U1.26 (IO2_3)
- net Sw 30: now also U1.36 (IO3_0)
- net Sw 31: now also U1.21 (IO1_7)
- net Sw 32: now also U1.20 (IO1_6)
- net Sw 36: now also SW37.2 (Sw2); no longer SW36.2 (Sw2)
- net Sw 37: now also SW36.2 (Sw2); no longer SW37.2 (Sw2)
- net Sw 4: now also U1.14 (IO1_1)
- net Sw 8: now also U1.43 (IO3_6)
- net Sw 9: now also U1.32 (IO2_5)
- net at SW3.DOUT: now also SW10.DIN; no longer SW4.DIN
- net at SW27.DOUT: now also SW20.DIN; no longer SW28.DIN
- net at SW29.DIN: now also SW22.DOUT; no longer SW28.DOUT
- net at SW17.DOUT: now also SW24.DIN; no longer SW18.DIN
- net at SW19.DIN: now also SW12.DOUT; no longer SW18.DOUT
- net at SW10.DOUT: now also SW17.DIN; no longer SW11.DIN
- net at SW12.DIN: now also SW5.DOUT; no longer SW11.DOUT
- net at SW26.DOUT: now also SW33.DIN; no longer SW27.DIN
- net at SW35.DOUT: now also SW38.DIN; no longer SW36.DIN
- net at SW37.DIN: now also SW33.DOUT; no longer SW36.DOUT
- net at SW1.DOUT: now also SW8.DIN; no longer SW2.DIN
- net at LED31.2 (DIN): now also LED36.4 (DOUT); no longer LED30.4 (DOUT)
- net at SW6.DIN: now also SW13.DOUT; no longer SW5.DOUT
- net at SW9.DOUT: now also SW2.DIN; no longer SW10.DIN
- net at SW23.DOUT: now also SW16.DIN; no longer SW24.DIN
- net at SW24.DOUT: now also SW31.DIN; no longer SW25.DIN
- net at SW32.DOUT: now also SW25.DIN; no longer SW33.DIN
- net at SW15.DOUT: now also SW22.DIN; no longer SW16.DIN
- net at SW16.DOUT: now also SW9.DIN; no longer SW17.DIN
- net at SW30.DOUT: now also SW23.DIN; no longer SW31.DIN
- net at SW7.DOUT: now also SW14.DIN; no longer SW8.DIN
- net at SW37.DOUT: now also SW27.DIN; no longer SW38.DIN
- net at SW26.DIN: now also SW19.DOUT; no longer SW25.DOUT
- net at SW15.DIN: now also SW8.DOUT; no longer SW14.DOUT
- net at SW21.DOUT: now also SW28.DIN; no longer SW22.DIN
- net at SW13.DIN: now also SW20.DOUT; no longer SW12.DOUT
- net at SW34.DIN: now also SW36.DOUT; no longer SW33.DOUT
- net at SW21.DIN: now also SW14.DOUT; no longer SW20.DOUT
- new net: LED34.4 (DOUT), LED35.2 (DIN)
- new net: LED35.4 (DOUT), LED36.2 (DIN)
- new net: LED30.4 (DOUT), LED32.2 (DIN)
- new net: LED32.4 (DOUT), LED33.2 (DIN)
- new net: LED33.4 (DOUT), LED34.2 (DIN)
- new net: SW11.DOUT, SW4.DIN
- new net: U3.11 (VSS), U3.23 (VSS), U3.34 (VSS), U3.39 (VSS), U3.51 (VSS), U3.6 (VSS)
- new net: U3.18 (VDD), U3.46 (VDD)
- new net: SW28.DOUT, SW36.DIN
- new net: SW11.DIN, SW18.DOUT
- new net: SW18.DIN, SW25.DOUT
Other:
- moved on the sheet: AE1, BT1, C1, LED31, P1, P10, P11, P2, P3, P4, P5, P6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

Commit message: syncing to 3.2.25
Parts:
- removed BT1: BATTERY-18650, Batteries:BATTERY_18650-HOLDER, symbol SparkFun-Batteries:BATTERY-18650
- removed Rs1, Rs10, Rs11, Rs12, Rs2, Rs3, Rs4, Rs5, Rs6, Rs7, Rs8, Rs9: 220Ω, Resistor_SMD:R_0805_2012Metric_Pad1.20x1.40mm_HandSolder, symbol SparkFun-Resistors:RESISTORAXIAL-0.3-KIT
- removed U1, U2, U3: PCA9505DGG,118, PCA9505DGG_118:SOP50P810X120-56N, symbol PCA9505DGG_118:PCA9505DGG,118
- added CA1, CA2: Cap_Array_2x4, Custom:Capacitor Array 2x4, symbol Custom:Cap_Array_2x4
- added RA0, RA1, RA2, RA3: CAT16A_Resistor_Array, Custom:CAT16A-LF, symbol Custom:CAT16A_Resistor_Array
- added RA5, RA6, RA7, RA8: Resistor_Array, Custom:CAT10A Resistor Array, symbol Custom:Resistor_Array
- added U1, U2, U3, U5: PCA9555PW, SOP65P640X110-24N:SOP65P640X110-24N, symbol PCA9555PW:PCA9555PW
- S1, S2, S3, S4: footprint Switches:ENCODER_LED_3 -> Custom:LED Encoder Cutout
Connections:
- net +5V: now also RA5.1, RA5.2, RA6.1, RA6.2, RA7.1, RA7.2, RA8.1, RA8.2
- net GND: now also CA1.1, CA1.1, CA1.1, CA1.1, CA2.1, CA2.1, CA2.1, CA2.1
- net Rot 0 A: now also CA2.2, RA8.1; no longer S1.A
- net Rot 0 B: now also CA2.2, RA8.1; no longer S1.B
- net Rot 0 G: now also RA0.2
- net Rot 0 R: now also RA0.2
- net Rot 0 U: now also RA0.2
- net Rot 1 A: now also CA2.2, RA6.1; no longer S2.A
- net Rot 1 B: now also CA2.2, RA6.1; no longer S2.B
- net Rot 1 G: now also RA1.2
- net Rot 1 R: now also RA1.2
- net Rot 1 U: now also RA1.2
- net Rot 2 A: now also CA1.2, RA7.1; no longer S3.A
- net Rot 2 B: now also CA1.2, RA7.1; no longer S3.B
- net Rot 2 G: now also RA2.2
- net Rot 2 R: now also RA2.2
- net Rot 2 U: now also RA2.2
- net Rot 3 A: now also CA1.2, RA5.1; no longer S4.A
- net Rot 3 B: now also CA1.2, RA5.1; no longer S4.B
- net Rot 3 G: now also RA3.2
- net Rot 3 R: now also RA3.2
- net Rot 3 U: now also RA3.2
- net SCL: now also U1.22 (SCL), U2.22 (SCL), U3.22 (SCL), U5.22 (SCL)
- net SDA: now also U1.23 (SDA), U2.23 (SDA), U3.23 (SDA), U5.23 (SDA)
- net at S3.1 (-R): now also RA2.1
- net at S2.1 (-R): now also RA1.1
- net at S3.4 (-B): now also RA2.1
- net at S1.2 (-G): now also RA0.1
- net at S1.4 (-B): now also RA0.1
- net at S4.2 (-G): now also RA3.1
- net at S4.1 (-R): now also RA3.1
- net at S4.4 (-B): now also RA3.1
- net at S3.2 (-G): now also RA2.1
- net at S1.1 (-R): now also RA0.1
- net at S2.2 (-G): now also RA1.1
- net at S2.4 (-B): now also RA1.1
- net Bat +: no longer names the net of U4.22 (Batt_+)
- net Bat -: no longer names the net of U4.21 (Batt-)
- new net: RA7.1, RA7.2, S3.B
- new net: RA8.2, RA8.2, S1.A
- new net: RA8.1, RA8.2, S1.B
- new net: RA6.2, RA6.2, S2.A
- new net: RA5.1, RA5.2, S4.B
- new net: RA5.2, RA5.2, S4.A
- new net: RA6.1, RA6.2, S2.B
- new net: RA7.2, RA7.2, S3.A
Other:
- moved on the sheet: J1, OLED1, RSW1, RSW2
